File: PESTFlex/PESTFlex.kicad_sch (KiCad schematic)
At the start: 24 parts, among them J1 Conn_01x07

Commit message: Finalized PCBs for fabrication
Parts:
- D1, D10, D11, D2, D3, D4, D5, D6, D7, D8, D9: footprint (none) -> Touchstone:ES2A-L Diode
- J1: footprint (none) -> Touchstone:Flex2Driver
- renumbered L2 to L1, L11 to L10, L12 to L11, L1 to L12, L3 to L2, L4 to L3, L5 to L4, L6 to L5, L7 to L6, L8 to L7, L9 to L8, L10 to L9
Connections:
- net A0: now also J1.7 (Pin_7); no longer J1.1 (Pin_1)
- net B0: now also J1.1 (Pin_1); no longer J1.2 (Pin_2)
- net X0: now also J1.2 (Pin_2); no longer J1.3 (Pin_3)
- net X1: now also J1.3 (Pin_3); no longer J1.4 (Pin_4)
- net X2: now also J1.4 (Pin_4); no longer J1.5 (Pin_5)
- net Y1: now also J1.5 (Pin_5); no longer J1.7 (Pin_7)
Other:
- moved on the sheet: L12
