File: TrackRing/TrackRing.kicad_sch (KiCad schematic)
At the start: 7 parts, among them J1 Conn_01x04, U1 TLV493D-A1B6

Commit message: Finalized PCBs for fabrication
Parts:
- added D1: LED, LED_SMD:LED_0603_1608Metric, symbol Device:LED
- added R98: 500, Resistor_SMD:R_0402_1005Metric, symbol Device:R
Connections:
- net GND: now also R98.2
- net VCC: now also D1.2 (A)
- new net: D1.1 (K), R98.1
Changed lines of the file:
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@@
+    (effects (font (size 1.27 1.27)) (justify right bottom))
+  )
+  (label "VCC" (at 38.735 55.88 180) (fields_autoplaced)
     (effects (font (size 1.27 1.27)) (justify right bottom))
   )
@@
   (label "VCC" (at 27.305 33.655 180) (fields_autoplaced)
     (effects (font (size 1.27 1.27)) (justify right bottom))
+  )
+  (symbol (lib_id "power:GND") (at 53.975 55.88 90) (unit 1)
+    (in_bom yes) (on_board yes) (dnp no) (fields_autoplaced)
+    (property "Reference" "#PWR04" (at 60.325 55.88 0)
+      (effects (font (size 1.27 1.27)) hide)
+    )
+    (property "Value" "GND" (at 57.785 56.515 90)
+      (effects (font (size 1.27 1.27)) (justify right))
+    )
+    (property "Footprint" "" (at 53.975 55.88 0)
+      (effects (font (size 1.27 1.27)) hide)
+    )
+    (property "Datasheet" "" (at 53.975 55.88 0)
+      (effects (font (size 1.27 1.27)) hide)
+    )
+    (pin "1")
+    (instances
+      (project "TrackRing"
+        (path "/1a22a45d-0453-4b94-9e49-dc92af99da64"
+          (reference "#PWR04") (unit 1)
+        )
+      )
+      (project "BusChain"
+        (path "/a3c96221-c538-4784-bbfe-f272329e4c12"
+          (reference "#PWR026") (unit 1)
+        )
+      )
+    )
   )
   (symbol (lib_id "Device:R") (at 59.055 33.655 0) (unit 1)
@@
     (pin "2")
     (instances
-      (project "Magnetic_Encoder"
+      (project "TrackRing"
         (path "/1a22a45d-0453-4b94-9e49-dc92af99da64"
           (reference "R3") (unit 1)
@@
     (pin "6")
     (instances
-      (project "Magnetic_Encoder"
+      (project "TrackRing"
         (path "/1a22a45d-0453-4b94-9e49-dc92af99da64"
           (reference "U1") (unit 1)
+        )
+      )
+    )
+  )
+  (symbol (lib_id "Device:R") (at 50.165 55.88 90) (unit 1)
+    (in_bom yes) (on_board yes) (dnp no) (fields_autoplaced)
+    (property "Reference" "R98" (at 50.165 51.435 90)
+      (effects (font (size 1.27 1.27)))
+    )
+    (property "Value" "500" (at 50.165 53.975 90)
+      (effects (font (size 1.27 1.27)))
+    )
+    (property "Footprint" "Resistor_SMD:R_0402_1005Metric" (at 50.165 57.658 90)
+      (effects (font (size 1.27 1.27)) hide)
+    )
+    (property "Datasheet" "~" (at 50.165 55.88 0)
+      (effects (font (size 1.27 1.27)) hide)
+    )
+    (pin "1")
+    (pin "2")
+    (instances
+      (project "PEST_Driver"
+        (path "/1312aa0a-e5d3-4b8d-ac4b-b6abdfb7d180"
+          (reference "R98") (unit 1)
+        )
+      )
+      (project "TrackRing"
+        (path "/1a22a45d-0453-4b94-9e49-dc92af99da64"
+          (reference "R5") (unit 1)
+        )
+      )
+      (project "BusChain"
+        (path "/a3c96221-c538-4784-bbfe-f272329e4c12"
+          (reference "R3") (unit 1)
         )
       )
@@
     (pin "1")
     (instances
-      (project "Magnetic_Encoder"
+      (project "TrackRing"
         (path "/1a22a45d-0453-4b94-9e49-dc92af99da64"
           (reference "#PWR03") (unit 1)
@@
     (pin "2")
     (instances
-      (project "Magnetic_Encoder"
+      (project "TrackRing"
         (path "/1a22a45d-0453-4b94-9e49-dc92af99da64"
           (reference "R2") (unit 1)
@@
     (pin "1")
     (instances
-      (project "Magnetic_Encoder"
+      (project "TrackRing"
         (path "/1a22a45d-0453-4b94-9e49-dc92af99da64"
           (reference "#PWR01") (unit 1)
@@
     (pin "2")
     (instances
-      (project "Magnetic_Encoder"
+      (project "TrackRing"
         (path "/1a22a45d-0453-4b94-9e49-dc92af99da64"
           (reference "R1") (unit 1)
@@
     (pin "2")
     (instances
-      (project "Magnetic_Encoder"
+      (project "TrackRing"
         (path "/1a22a45d-0453-4b94-9e49-dc92af99da64"
           (reference "R4") (unit 1)
@@
     (pin "4")
     (instances
-      (project "Magnetic_Encoder"
+      (project "TrackRing"
         (path "/1a22a45d-0453-4b94-9e49-dc92af99da64"
           (reference "J1") (unit 1)
@@
     )
   )
+  (symbol (lib_id "Device:LED") (at 42.545 55.88 180) (unit 1)
+    (in_bom yes) (on_board yes) (dnp no) (fields_autoplaced)
+    (property "Reference" "D1" (at 44.1325 49.53 0)
+      (effects (font (size 1.27 1.27)))
+    )
+    (property "Value" "LED" (at 44.1325 52.07 0)
+      (effects (font (size 1.27 1.27)))
+    )
+    (property "Footprint" "LED_SMD:LED_0603_1608Metric" (at 42.545 55.88 0)
+      (effects (font (size 1.27 1.27)) hide)
+    )
+    (property "Datasheet" "~" (at 42.545 55.88 0)
+      (effects (font (size 1.27 1.27)) hide)
+    )
+    (pin "1")
+    (pin "2")
+    (instances
+      (project "PEST_Driver"
+        (path "/1312aa0a-e5d3-4b8d-ac4b-b6abdfb7d180"
+          (reference "D1") (unit 1)
+        )
+      )
+      (project "TrackRing"
+        (path "/1a22a45d-0453-4b94-9e49-dc92af99da64"
+          (reference "D1") (unit 1)
+        )
+      )
+      (project "BusChain"
+        (path "/a3c96221-c538-4784-bbfe-f272329e4c12"
+          (reference "D1") (unit 1)
+        )
+      )
+    )
+  )
   (symbol (lib_id "Device:C") (at 76.835 24.13 0) (unit 1)
     (in_bom yes) (on_board yes) (dnp no) (fields_autoplaced)
@@
     (pin "2")
     (instances
-      (project "Magnetic_Encoder"
+      (project "TrackRing"
         (path "/1a22a45d-0453-4b94-9e49-dc92af99da64"
           (reference "C1") (unit 1)
@@
     (pin "1")
     (instances
-      (project "Magnetic_Encoder"
+      (project "TrackRing"
         (path "/1a22a45d-0453-4b94-9e49-dc92af99da64"
           (reference "#PWR02") (unit 1)
