File: BusChain/BusChain.kicad_pcb (KiCad board)
At the start: 2 copper layers, 48 x 16 mm, 27 parts, among them J1 Conn_01x04, J10 Conn_01x04, J2 Conn_01x04, J3 Conn_01x04, J4 Conn_01x04, J5 Conn_01x04, J6 Conn_01x04, J7 Conn_01x04, J8 Conn_01x04, J9 Conn_01x04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

Commit message: Final fabrication checks
Parts:
- removed D2: LED, LED_SMD:LED_0603_1608Metric
- removed R4: 500, Resistor_SMD:R_0402_1005Metric
- moved R3 0.85 mm to (66.0, 33.2)
- moved D1 0.85 mm to (63.3, 33.2)
Routing:
- net /SCL: track 51.7 -> 46.7 mm
- net /VCC: track 101.2 -> 97.1 mm
- net Net-(D2-K): track 1.45 -> 0.00 mm
- net GND: track 9.97 -> 9.00 mm, vias 9 -> 8
Other:
- board text added: "VCC"
