File: BusChain/BusChain.kicad_sch (KiCad schematic)
At the start: 27 parts, among them J1 Conn_01x04, J10 Conn_01x04, J2 Conn_01x04, J3 Conn_01x04, J4 Conn_01x04, J5 Conn_01x04, J6 Conn_01x04, J7 Conn_01x04, J8 Conn_01x04, J9 Conn_01x04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

Commit message: Final fabrication checks
Parts:
- removed D2: LED, LED_SMD:LED_0603_1608Metric, symbol Device:LED
- removed R99: 500, Resistor_SMD:R_0402_1005Metric, symbol Device:R
Changed lines of the file:
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@@
-    (effects (font (size 1.27 1.27)) (justify right bottom))
-  )
-  (label "SCL" (at 86.36 142.875 180) (fields_autoplaced)
     (effects (font (size 1.27 1.27)) (justify right bottom))
   )
@@
     (effects (font (size 1.27 1.27)) (justify left bottom))
   )
-  (symbol (lib_id "Device:R") (at 97.79 142.875 90) (unit 1)
-    (in_bom yes) (on_board yes) (dnp no) (fields_autoplaced)
-    (property "Reference" "R99" (at 97.79 138.43 90)
-      (effects (font (size 1.27 1.27)))
-    )
-    (property "Value" "500" (at 97.79 140.97 90)
-      (effects (font (size 1.27 1.27)))
-    )
-    (property "Footprint" "Resistor_SMD:R_0402_1005Metric" (at 97.79 144.653 90)
-      (effects (font (size 1.27 1.27)) hide)
-    )
-    (property "Datasheet" "~" (at 97.79 142.875 0)
-      (effects (font (size 1.27 1.27)) hide)
-    )
-    (pin "1")
-    (pin "2")
-    (instances
-      (project "PEST_Driver"
-        (path "/1312aa0a-e5d3-4b8d-ac4b-b6abdfb7d180"
-          (reference "R99") (unit 1)
-        )
-      )
-      (project "BusChain"
-        (path "/a3c96221-c538-4784-bbfe-f272329e4c12"
-          (reference "R4") (unit 1)
-        )
-      )
-    )
-  )
   (symbol (lib_id "power:GND") (at 147.955 136.525 0) (unit 1)
     (in_bom yes) (on_board yes) (dnp no) (fields_autoplaced)
@@
         (path "/a3c96221-c538-4784-bbfe-f272329e4c12"
           (reference "#PWR018") (unit 1)
-        )
-      )
-    )
-  )
-  (symbol (lib_id "power:GND") (at 101.6 142.875 90) (unit 1)
-    (in_bom yes) (on_board yes) (dnp no) (fields_autoplaced)
-    (property "Reference" "#PWR06" (at 107.95 142.875 0)
-      (effects (font (size 1.27 1.27)) hide)
-    )
-    (property "Value" "GND" (at 105.41 143.51 90)
-      (effects (font (size 1.27 1.27)) (justify right))
-    )
-    (property "Footprint" "" (at 101.6 142.875 0)
-      (effects (font (size 1.27 1.27)) hide)
-    )
-    (property "Datasheet" "" (at 101.6 142.875 0)
-      (effects (font (size 1.27 1.27)) hide)
-    )
-    (pin "1")
-    (instances
-      (project "BusChain"
-        (path "/a3c96221-c538-4784-bbfe-f272329e4c12"
-          (reference "#PWR06") (unit 1)
         )
       )
@@
         )
       )
-    )
-  )
-  (symbol (lib_id "Device:LED") (at 90.17 142.875 180) (unit 1)
-    (in_bom yes) (on_board yes) (dnp no) (fields_autoplaced)
-    (property "Reference" "D2" (at 91.7575 136.525 0)
-      (effects (font (size 1.27 1.27)))
-    )
-    (property "Value" "LED" (at 91.7575 139.065 0)
-      (effects (font (size 1.27 1.27)))
-    )
-    (property "Footprint" "LED_SMD:LED_0603_1608Metric" (at 90.17 142.875 0)
-      (effects (font (size 1.27 1.27)) hide)
-    )
-    (property "Datasheet" "~" (at 90.17 142.875 0)
-      (effects (font (size 1.27 1.27)) hide)
-    )
-    (pin "1")
-    (pin "2")
-    (instances
-      (project "PEST_Driver"
-        (path "/1312aa0a-e5d3-4b8d-ac4b-b6abdfb7d180"
-          (reference "D2") (unit 1)
-        )
-      )
-      (project "BusChain"
-        (path "/a3c96221-c538-4784-bbfe-f272329e4c12"
-          (reference "D2") (unit 1)
-        )
-      )
