File: AS5600/AS5600.kicad_pcb (KiCad board)
At the start: 2 copper layers, 15 x 15 mm, 10 parts, among them IC1 AS5600-ASOT, J1 Conn_01x02, J2 Conn_01x04

Commit message: Fixed pin header orientation and added silkscreen
Parts:
- J1: footprint Connector_PinHeader_2.54mm:PinHeader_1x02_P2.54mm_Vertical -> Connector_PinHeader_2.54mm:PinHeader_1x02_P2.54mm_Horizontal
- J2: footprint Connector_PinHeader_2.54mm:PinHeader_1x04_P2.54mm_Vertical -> Connector_PinHeader_2.54mm:PinHeader_1x04_P2.54mm_Horizontal
- moved J1 1.25 mm to (24.5, 23.2)
- moved J2 1.25 mm to (22.0, 31.8)
Routing:
- net /SCL: track 9.23 -> 8.71 mm
- net /SDA: track 8.33 -> 8.83 mm
Other:
- board text added: "MagEncode 1.0"
- board text added: "©CGR"
