File: Hydra_Driver_Sheild/Hydra_Driver_Sheild.kicad_pcb (KiCad board)
At the start: 2 copper layers, 69 x 42 mm, 104 parts, among them IC1 ESP32-S3-WROOM-1-N4, IC2 DRV8313RHHR, IC3 DRV8313RHHR, J1 USB4105-GF-A, J10 Conn_01x03, J11 Conn_01x04, J12 Conn_01x03, J13 Conn_01x02, J2 Conn_01x02, J3 Conn_01x06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

Commit message: Finished hydra shield version
Parts:
- removed J13, J2: Conn_01x02, TerminalBlock:TerminalBlock_MaiXu_MX126-5.0-02P_1x02_P5.00mm
- removed J3: Conn_01x06, Connector_PinSocket_2.54mm:PinSocket_1x06_P2.54mm_Horizontal
- removed J7: Conn_01x02, Connector_PinSocket_2.54mm:PinSocket_1x02_P2.54mm_Vertical
- removed J9: Conn_01x06, Connector_PinHeader_2.54mm:PinHeader_1x06_P2.54mm_Horizontal
- J10, J4, J8: footprint Connector_PinSocket_2.54mm:PinSocket_1x03_P2.54mm_Vertical -> Connector_PinHeader_2.54mm:PinHeader_1x03_P2.54mm_Vertical; moved to B.Cu
- J11, J12, J5, J6: moved to F.Cu
- turned J10 to -90 degrees
- turned J11 to 90 degrees
- turned J12 to 90 degrees
- turned J4 to -90 degrees
- turned J5 to 90 degrees
- turned J6 to 90 degrees
- turned J8 to -90 degrees
Connections:
- J10 pad 1: /LOOP2 -> /MOSI
- J4 pad 1: /LOOP1 -> /MISO
Routing:
- net /LOOP1: track 45.5 -> 0.00 mm
- net VMOT: track 129.2 -> 118.2 mm
- net +5V: track 82.0 -> 73.2 mm
- net /LOOP2: track 7.44 -> 0.00 mm
- net /MISO: track 24.4 -> 29.5 mm, vias 1 -> 2
- net /MOSI: track 30.2 -> 27.2 mm
- net /SCL1: track 29.2 -> 27.8 mm
- net /CLK: track 52.6 -> 52.1 mm, vias 2 -> 3
- net /CS: track 44.1 -> 44.0 mm, vias 3 -> 4
Other:
- board text added: "HYDRA SHIELD"
- board text removed: "HYDRA"
- board text removed: "L1"
- board text removed: "L2"
- board text removed: "NSHIELD"
