File: Hydra_Driver_Shield/Hydra_Driver_Shield.kicad_pcb (KiCad board)
At the start: 2 copper layers, 69 x 42 mm, 99 parts, among them IC1 ESP32-S3-WROOM-1-N4, IC2 DRV8313RHHR, IC3 DRV8313RHHR, J1 USB4105-GF-A, J10 Conn_01x03, J11 Conn_01x04, J12 Conn_01x03, J4 Conn_01x03, J5 Conn_01x04, J6 Conn_01x03, J8 Conn_01x03, SW1 SW_SPST, SW2 SW_SPST, U1 USBLC6-2SC6, U2 MIC5365-3.3YC5, U3 74HC32, U4 INA199xxDCK, U5 INA199xxDCK, U6 74HC32, U7 INA199xxDCK, U8 INA199xxDCK

Commit message: Finished updating shield board with changes
Parts:
- removed the C23 at (44.3, 9.50)
- removed C34: 0.1u, Capacitor_SMD:C_0402_1005Metric
- removed the R10 at (30.0, 38.2)
- removed the R11 at (44.0, 24.5)
- removed the R12 at (46.0, 21.5)
- removed the R13 at (47.2, 21.5)
- removed the R14 at (44.8, 18.5)
- removed the R15 at (48.5, 18.5)
- removed the R16 at (48.0, 9.50)
- removed R24, R25, R26, R27, R28, R29: 3.3k, Resistor_SMD:R_0402_1005Metric
- removed the REF** at (66.5, 2.50)
- removed the REF** at (2.50, 30.2)
- removed the REF** at (66.5, 39.5)
- removed the U3 at (47.2, 13.8)
- removed the U6 at (60.6, 13.7)
- added R8: 10k, Resistor_SMD:R_0402_1005Metric, F.Cu at (26.7, 41.2)
- added REF**: MountingHole_2.2mm_M2, MountingHole:MountingHole_2.2mm_M2, F.Cu at (39.4, 39.4)
- added REF**: MountingHole_2.2mm_M2, MountingHole:MountingHole_2.2mm_M2, F.Cu at (50.2, 10.0)
- added REF**: MountingHole_2.2mm_M2, MountingHole:MountingHole_2.2mm_M2, F.Cu at (2.60, 30.0)
- J3: renamed from J5; footprint Connector_PinHeader_2.54mm:PinHeader_1x04_P2.54mm_Vertical -> Connector_PinHeader_2.54mm:PinHeader_1x04_P2.54mm_Horizontal; moved to B.Cu
- J4: renamed from J6; footprint Connector_PinHeader_2.54mm:PinHeader_1x03_P2.54mm_Vertical -> Connector_PinHeader_2.54mm:PinHeader_1x03_P2.54mm_Horizontal; moved to B.Cu
- J7: renamed from J11; footprint Connector_PinHeader_2.54mm:PinHeader_1x04_P2.54mm_Vertical -> Connector_PinHeader_2.54mm:PinHeader_1x04_P2.54mm_Horizontal; moved to B.Cu
- J8: renamed from J12; footprint Connector_PinHeader_2.54mm:PinHeader_1x03_P2.54mm_Vertical -> Connector_PinHeader_2.54mm:PinHeader_1x03_P2.54mm_Horizontal; moved to B.Cu
- U2: value MIC5365-3.3YC5 -> MIC5504-3.3YM5-TR; footprint Package_TO_SOT_SMD:SOT-353_SC-70-5 -> Touchstone:SOT-23-5_MC_MCH
- moved C11 36.9 mm to (41.8, 2.42)
- moved C12 36.9 mm to (43.2, 2.45)
- moved C8 36.9 mm to (50.0, 2.45)
- moved C9 36.9 mm to (51.5, 2.38)
- moved U2 36.7 mm to (46.6, 2.70)
- moved C25 25.0 mm to (48.3, 14.0), turned to 180 degrees
- moved R20 24.8 mm to (42.3, 16.0), turned to 180 degrees
- moved D5 24.6 mm to (42.8, 13.2), turned to 180 degrees
- moved R22 24.5 mm to (43.8, 15.5), turned to 90 degrees
- moved R18 23.6 mm to (42.2, 11.7), turned to 0 degrees
- moved R19 23.4 mm to (42.2, 14.7), turned to 0 degrees
- moved C32 23.2 mm to (45.2, 16.0), turned to 180 degrees
- moved C31 22.7 mm to (50.0, 15.5), turned to 180 degrees
- moved C29 22.4 mm to (47.5, 16.0), turned to 180 degrees
- moved R23 21.3 mm to (45.5, 13.2), turned to 0 degrees
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- renumbered C24 to C23, C25 to C24, C26 to C25, C27 to C26, C28 to C27, C29 to C28, C30 to C29, C31 to C30, C32 to C31, C33 to C32, J4 to J2, J8 to J5, J10 to J6, R17 to R10, R18 to R11, R19 to R12, R20 to R13, R21 to R14, R22 to R15, R23 to R16, R30 to R17, R31 to R18, R32 to R19, R33 to R20, R34 to R21, R35 to R22, R36 to R23, U4 to U3, U5 to U4, U7 to U5, U8 to U6
Connections:
- net /IN1HA renamed /IN1A
- net /IN1HB renamed /IN1B
- net /IN2HA renamed /IN2A
- net /IN2HB renamed /IN2B
- net /IN3HA renamed /IN3A
- net /IN3HB renamed /IN3B
- IC1 pad 15: /IN1LA -> /EN1A
- IC1 pad 17: /IN2LA -> /EN2A
- IC1 pad 19: /IN3LA -> /EN3A
- IC1 pad 24: /IN1LB -> /EN1B
- IC1 pad 26: /IN2LB -> /EN2B
- IC1 pad 29: /IN3LB -> /EN3B
- IC1 pad 30: /SDA2 -> /SDA1
- IC1 pad 31: /SCL2 -> /SCL1
- IC1 pad 32: /SDA1 -> /SDA2
- IC1 pad 33: /SCL1 -> /SCL2
- IC2 pad 1: /Driver_Unit/EN1 -> /EN1A
- IC2 pad 33: /Driver_Unit/EN3 -> /EN3A
- IC2 pad 35: /Driver_Unit/EN2 -> /EN2A
- IC3 pad 1: /Driver_Unit1/EN1 -> /EN1B
- IC3 pad 33: /Driver_Unit1/EN3 -> /EN3B
- IC3 pad 35: /Driver_Unit1/EN2 -> /EN2B
Routing:
- net /IN2LB: track 33.5 -> 0.00 mm
- net /IN3LB: track 32.1 -> 0.00 mm, vias 2 -> 0
- net /IN1LB: track 31.5 -> 0.00 mm
- net /IN2B: track 39.9 -> 10.2 mm
- net /IN1B: track 39.7 -> 11.1 mm
- net /IN3B: track 44.4 -> 15.9 mm, vias 2 -> 0
- net +3.3V: track 185.1 -> 158.4 mm, vias 7 -> 10
- net /IN3A: track 34.7 -> 13.1 mm
- net /IN3LA: track 21.3 -> 0.00 mm
- net VMOT: track 118.2 -> 97.3 mm
- net GND: track 105.7 -> 125.9 mm, vias 31 -> 42
- net /IN1LA: track 20.2 -> 0.00 mm
- net /SENSE2A: track 25.4 -> 44.1 mm
- net /SENSE1B: track 34.6 -> 52.6 mm
- net /SENSE2B: track 45.4 -> 62.1 mm
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Other:
- board size 69 x 42 mm -> 59.2 x 42 mm
- board text added: "FAULT"
- board text added: "I2C1"
- board text added: "I2C2"
- board text added: "L1"
- board text added: "L2"
- board text added: "SCL"
- board text added: "SDA"
- board text removed: "SCL1"
- board text removed: "SCL2"
- board text removed: "SDA1"
- board text removed: "SDA2"
