File: Hydra_Driver_Shield/Hydra_Driver_Shield.kicad_pcb (KiCad board)
At the start: 2 copper layers, 59.2 x 42 mm, 83 parts, among them IC1 ESP32-S3-WROOM-1-N4, IC2 DRV8313RHHR, IC3 DRV8313RHHR, J1 USB4105-GF-A, J2 Conn_01x03, J3 Conn_01x04, J4 Conn_01x03, J5 Conn_01x03, J6 Conn_01x03, J7 Conn_01x04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

Commit message: Consolidated pullup resistors to 10k
Parts:
- R11, R12, R13, R15, R18, R19, R20, R22: value 3.3k -> 10k
