File: Hydra_Driver_Shield/Hydra_Driver_Shield.kicad_sch (KiCad schematic)
At the start: 38 parts, among them IC1 ESP32-S3-WROOM-1-N4, J1 USB4105-GF-A, J10 Conn_01x03, J11 Conn_01x04, J12 Conn_01x03, J4 Conn_01x03, J5 Conn_01x04, J6 Conn_01x03, J8 Conn_01x03, SW1 SW_SPST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

Commit message: Finished updating shield board with changes
Parts:
- removed R10: 10k, Resistor_SMD:R_0402_1005Metric, symbol Device:R
- removed U2: MIC5365-3.3YC5, Package_TO_SOT_SMD:SOT-353_SC-70-5, symbol Regulator_Linear:MIC5365-3.3YC5
- added U2: MIC5504-3.3YM5-TR, Touchstone:SOT-23-5_MC_MCH, symbol MIC5504:MIC5504-3.3YM5-TR
- J3: renamed from J5; footprint Connector_PinHeader_2.54mm:PinHeader_1x04_P2.54mm_Vertical -> Connector_PinHeader_2.54mm:PinHeader_1x04_P2.54mm_Horizontal
- J4: renamed from J6; footprint Connector_PinHeader_2.54mm:PinHeader_1x03_P2.54mm_Vertical -> Connector_PinHeader_2.54mm:PinHeader_1x03_P2.54mm_Horizontal
- J7: renamed from J11; footprint Connector_PinHeader_2.54mm:PinHeader_1x04_P2.54mm_Vertical -> Connector_PinHeader_2.54mm:PinHeader_1x04_P2.54mm_Horizontal
- J8: renamed from J12; footprint Connector_PinHeader_2.54mm:PinHeader_1x03_P2.54mm_Vertical -> Connector_PinHeader_2.54mm:PinHeader_1x03_P2.54mm_Horizontal
- renumbered J4 to J2, J8 to J5, J10 to J6
Connections:
- net +3.3V: now also U2.5 (VOUT)
- net +5V: now also U2.1 (VIN), U2.3 (EN)
- net GND: now also U2.2 (GND)
- net SCL1: now also IC1.31 (IO38); no longer IC1.33 (IO40)
- net SCL2: now also IC1.33 (IO40); no longer IC1.31 (IO38)
- net SDA1: now also IC1.30 (IO37); no longer IC1.32 (IO39)
- net SDA2: now also IC1.32 (IO39); no longer IC1.30 (IO37)
- net IN1HA renamed IN1A
- net IN1HB renamed IN1B
- net IN1LA renamed EN1A
- net IN1LB renamed EN1B
- net IN2HA renamed IN2A
- net IN2HB renamed IN2B
- net IN2LA renamed EN2A
- net IN2LB renamed EN2B
- net IN3HA renamed IN3A
- net IN3HB renamed IN3B
- net IN3LA renamed EN3A
- net IN3LB renamed EN3B
Other:
- sheet Driver_Unit ports: added EN1, EN2, EN3, IN1, IN2, IN3; removed IN1H, IN1L, IN2H, IN2L, IN3H, IN3L
- sheet Driver_Unit1 ports: added EN1, EN2, EN3, IN1, IN2, IN3; removed IN1H, IN1L, IN2H, IN2L, IN3H, IN3L
- moved on the sheet: C11, C12, C8, C9, D2, D3, J2, J3, J4, J6, J7, J8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
